Commit message: it can use but have some wrong

File: AI_pkg/robot_arm/arm_ver6/test_abb_4600.urdf (robot description, URDF)
Before this commit: robot robot_ver6, 9 links, 8 joints
Links:
- removed link Component8_1
- removed link Component9_1
- removed link Component9_Mirror__1
- removed link base_link2_v2_1
- removed link grap2_v2_1
- removed link link3_v1_1
- removed link link4_v1_1
- removed link rotate_v2_v1_1
- added link robot_ver7_grap2_2_v1_1, mass 0.040626783640930315; collision mesh filename=package://test_description/meshes/robot_ver7_grap2_2_v1_1.s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 scale=0.001 0.001 0.001; visual mesh filename=package://test_description/meshes/robot_ver7_grap2_2_v1_1.s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 scale=0.001 0.001 0.001
- added link robot_ver7_grap_1_v1_1, mass 0.04062678364093055; collision mesh filename=package://test_description/meshes/robot_ver7_grap_1_v1_1.stl scale=0.001 0.001 0.001; visual mesh filename=package://test_description/meshes/robot_ver7_grap_1_v1_1.stl scale=0.001 0.001 0.001
- added link robot_ver7_grap_1_v1__1__1, mass 0.04062678364093055; collision mesh filename=package://test_description/meshes/robot_ver7_grap_1_v1__1__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 scale=0.001 0.001 0.001; visual mesh filename=package://test_description/meshes/robot_ver7_grap_1_v1__1__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 scale=0.001 0.001 0.001
- added link robot_ver7_grap_2_v1_1, mass 0.040626783640931016; collision mesh filename=package://test_description/meshes/robot_ver7_grap_2_v1_1.stl scale=0.001 0.001 0.001; visual mesh filename=package://test_description/meshes/robot_ver7_grap_2_v1_1.stl scale=0.001 0.001 0.001
- added link robot_ver7_link_1_v1_1, mass 0.8724221516718077; collision mesh filename=package://test_description/meshes/robot_ver7_link_1_v1_1.stl scale=0.001 0.001 0.001; visual mesh filename=package://test_description/meshes/robot_ver7_link_1_v1_1.stl scale=0.001 0.001 0.001
- added link robot_ver7_link_2_v1_1, mass 1.7894494256516231; collision mesh filename=package://test_description/meshes/robot_ver7_link_2_v1_1.stl scale=0.001 0.001 0.001; visual mesh filename=package://test_description/meshes/robot_ver7_link_2_v1_1.stl scale=0.001 0.001 0.001
- added link robot_ver7_link_3_v1_1, mass 2.3011672222568844; collision mesh filename=package://test_description/meshes/robot_ver7_link_3_v1_1.stl scale=0.001 0.001 0.001; visual mesh filename=package://test_description/meshes/robot_ver7_link_3_v1_1.stl scale=0.001 0.001 0.001
- added link robot_ver7_link_4_v1_1, mass 0.1836674229836166; collision mesh filename=package://test_description/meshes/robot_ver7_link_4_v1_1.stl scale=0.001 0.001 0.001; visual mesh filename=package://test_description/meshes/robot_ver7_link_4_v1_1.stl scale=0.001 0.001 0.001
- link base_link: mass 1.6067306789990294 -> 1.6067306789990348; geometry collision mesh filename=package://test_description/meshes/base_link.stl scale=0.001 0.001 0.001; visual mesh filename=package://test_description/meshes/base_link.stl scale=0.001 0.001 0.001
Joints:
- removed joint Revolute 2
- removed joint Revolute 3
- removed joint Revolute 4
- added joint Revolute 10: type continuous, parent robot_ver7_link_4_v1_1, child robot_ver7_grap_1_v1__1__1, origin xyz=0.043989 0.024541 -0.004982 rpy=0 0 0, axis 0.010462 0.999945 0.0
- added joint Revolute 11: type continuous, parent robot_ver7_link_4_v1_1, child robot_ver7_grap2_2_v1_1, origin xyz=0.039648 0.024587 0.019638 rpy=0 0 0, axis 0.010462 0.999945 0.0
- added joint Revolute 5: type revolute, parent robot_ver7_link_1_v1_1, child robot_ver7_link_2_v1_1, origin xyz=0.0 0.0 0.070342 rpy=0 0 0, axis -0.010462 -0.999945 -0.0, limit lower=0.0 upper=6.2831853 effort=100 velocity=100
- joint Revolute 1: axis 0.0 0.0 1.0 -> 0.0 -0.0 1.0; child base_link2_v2_1 -> robot_ver7_link_1_v1_1; limit (none) -> lower=0.0 upper=6.2831853 effort=100 velocity=100; origin xyz=2.989375 1.139525 0.122186 rpy=0 0 0 -> xyz=2.989375 1.116433 0.077907 rpy=0 0 0; type continuous -> revolute
- joint Revolute 6: axis -1.0 -0.0 -0.0 -> -0.010462 -0.999945 -0.0; child grap2_v2_1 -> robot_ver7_link_3_v1_1; limit (none) -> lower=0.0 upper=6.2831853 effort=100 velocity=100; origin xyz=-0.025 0.0125 0.0422 rpy=0 0 0 -> xyz=0.137769 -0.001442 0.164195 rpy=0 0 0; parent rotate_v2_v1_1 -> robot_ver7_link_2_v1_1; type continuous -> revolute
- joint Revolute 7: axis -1.0 -0.0 -0.0 -> 0.984754 -0.010303 0.173648; child Component8_1 -> robot_ver7_link_4_v1_1; limit (none) -> lower=0.0 upper=6.2831853 effort=100 velocity=100; origin xyz=-0.025 -0.0125 0.0422 rpy=0 0 0 -> xyz=0.230271 -0.002409 0.042126 rpy=0 0 0; parent rotate_v2_v1_1 -> robot_ver7_link_3_v1_1; type continuous -> revolute
- joint Revolute 8: axis 1.0 -0.0 0.0 -> -0.010462 -0.999945 -0.0; child Component9_1 -> robot_ver7_grap_1_v1_1; origin xyz=0.025 0.0125 0.0422 rpy=0 0 0 -> xyz=0.039125 -0.025411 0.019638 rpy=0 0 0; parent rotate_v2_v1_1 -> robot_ver7_link_4_v1_1
- joint Revolute 9: axis 1.0 0.0 0.0 -> -0.010462 -0.999945 -0.0; child Component9_Mirror__1 -> robot_ver7_grap_2_v1_1; origin xyz=0.025 -0.0125 0.0422 rpy=0 0 0 -> xyz=0.043466 -0.025456 -0.004982 rpy=0 0 0; parent rotate_v2_v1_1 -> robot_ver7_link_4_v1_1
